Commit message: Align camera orientation to gripper

File: mercury/_pybullet/assets/franka_panda/panda_suction.urdf (robot description, URDF)
Before this commit: robot panda, 13 links, 12 joints
Joints:
- joint link8_to_baseLink: origin xyz=0 0 0 rpy=0 0 0 -> xyz=0 0 0 rpy=0 0 0.785

File: mercury/_pybullet/assets/franka_panda/panda_suction.urdf.xacro (robot description, xacro)
@@ -4,5 +4,5 @@
   <xacro:include filename="suction/suction-base.urdf" />
   <joint name="link8_to_baseLink" type="fixed">
-    <origin rpy="0 0 0" xyz="0 0 0"/>
+    <origin rpy="0 0 ${ 3.14 / 4}" xyz="0 0 0"/>
     <parent link="panda_link8"/>
     <child link="baseLink"/>

Commit message: Add collision to panda_suction.urdf.xacro

File: mercury/_pybullet/assets/franka_panda/panda_suction.urdf (robot description, URDF)
Before this commit: robot panda, 13 links, 12 joints
Links:
- link baseLink: geometry collision mesh filename=suction/base.obj scale=0.001 0.001 0.001; visual mesh filename=suction/base.obj scale=0.001 0.001 0.001
- link midLink: geometry collision mesh filename=suction/mid.obj scale=0.001 0.001 0.001; visual mesh filename=suction/mid.obj scale=0.001 0.001 0.001
- link tipLink: geometry collision mesh filename=suction/tip.obj scale=0.001 0.001 0.001; visual mesh filename=suction/tip.obj scale=0.001 0.001 0.001

File: mercury/_pybullet/assets/franka_panda/suction/suction-base.urdf (robot description, URDF)
Before this commit: robot suction-base.urdf, 2 links, 1 joints
Links:
- link baseLink: geometry collision mesh filename=suction/base.obj scale=0.001 0.001 0.001; visual mesh filename=suction/base.obj scale=0.001 0.001 0.001
- link midLink: geometry collision mesh filename=suction/mid.obj scale=0.001 0.001 0.001; visual mesh filename=suction/mid.obj scale=0.001 0.001 0.001

File: mercury/_pybullet/assets/franka_panda/suction/suction-head.urdf (robot description, URDF)
Before this commit: robot suction-head.urdf, 2 links, 1 joints
Links:
- link tipLink: geometry collision mesh filename=suction/tip.obj scale=0.001 0.001 0.001; visual mesh filename=suction/tip.obj scale=0.001 0.001 0.001

Commit message: Fix origin of tipLink

File: mercury/_pybullet/assets/franka_panda/panda_suction.urdf (robot description, URDF)
Before this commit: robot panda, 13 links, 12 joints
Links:
- link tipLink: geometry collision cylinder length=0.028 radius=0.01; visual cylinder length=0.028 radius=0.01
Joints:
- joint tipJoint: origin xyz=0.0 0.0 0.029 rpy=0.0 0.0 0.0 -> xyz=0.0 0.0 0.043 rpy=0.0 0.0 0.0

File: mercury/_pybullet/assets/franka_panda/suction/suction-head.urdf (robot description, URDF)
Before this commit: robot suction-head.urdf, 2 links, 1 joints
Links:
- link tipLink: geometry collision cylinder length=0.028 radius=0.01; visual cylinder length=0.028 radius=0.01
Joints:
- joint tipJoint: origin xyz=0.0 0.0 0.029 rpy=0.0 0.0 0.0 -> xyz=0.0 0.0 0.043 rpy=0.0 0.0 0.0
