Commit message: Update table geometry

File: ros/mercury_panda/robots/scene/table.xacro (robot description, xacro)
@@ -15,5 +15,5 @@
       <visual>
         <geometry>
-          <box size="1.2 1.2 0.075"/>
+          <box size="1.0 1.3 0.05"/>
         </geometry>
         <material name="white"/>
@@ -21,5 +21,5 @@
       <collision>
         <geometry>
-          <box size="1.2 1.2 0.075"/>
+          <box size="1.0 1.3 0.05"/>
         </geometry>
       </collision>
