Commit message: Create drl dir in robots

File: ros/mercury_panda/robots/drl/suction.xacro (robot description, xacro)
@@ -18,5 +18,5 @@
       <visual>
         <geometry>
-          <mesh filename="package://mercury_panda/robots/meshes/visual/suction_mount.obj"/>
+          <mesh filename="package://mercury_panda/robots/drl/meshes/visual/suction_mount.obj"/>
         </geometry>
         <material name="black"/>
@@ -24,5 +24,5 @@
       <collision>
         <geometry>
-          <mesh filename="package://mercury_panda/robots/meshes/collision/suction_mount.obj"/>
+          <mesh filename="package://mercury_panda/robots/drl/meshes/collision/suction_mount.obj"/>
         </geometry>
       </collision>

File: ros/mercury_panda/robots/panda_reorient.urdf.xacro (robot description, xacro)
@@ -2,7 +2,7 @@
 <robot xmlns:xacro="http://www.ros.org/wiki/xacro" name="panda">
   <xacro:include filename="$(find franka_description)/robots/panda_arm.urdf.xacro"/>
-  <xacro:include filename="$(find mercury_panda)/robots/include/suction_gripper.xacro"/>
+  <xacro:include filename="$(find mercury_panda)/robots/drl/suction.xacro"/>
   <xacro:suction_gripper ns="panda" rpy="${pi} 0 ${-pi/4}" xyz="0 0 0.0065" connected_to="panda_link8"/>
-  <xacro:include filename="$(find mercury_panda)/robots/include/table.xacro"/>
+  <xacro:include filename="$(find mercury_panda)/robots/drl/table.xacro"/>
   <xacro:table ns="panda" rpy="0 0 0" xyz="0.68 0 0.0375" connected_to="panda_link0"/>
 </robot>
