Commit message: Fix reorientation for new robot model

File: mercury/_pybullet/robots/franka_panda/panda_reorient.urdf (robot description, URDF)
Before this commit: robot panda, 12 links, 11 joints
Links:
- removed link panda_table
Joints:
- removed joint panda_table_joint

File: mercury/_pybullet/robots/franka_panda/panda_reorient.urdf.xacro (robot description, xacro)
@@ -4,5 +4,5 @@
   <xacro:include filename="$(find mercury_panda)/robots/include/suction_gripper.xacro"/>
   <xacro:suction_gripper ns="panda" rpy="${pi} 0 ${-pi/4}" xyz="0 0 0.0065" connected_to="panda_link8"/>
-  <xacro:include filename="$(find mercury_panda)/robots/include/table.xacro"/>
-  <xacro:table ns="panda" rpy="0 0 0" xyz="0.68 0 0.0375" connected_to="panda_link0"/>
+  <!-- <xacro:include filename="$(find mercury_panda)/robots/include/table.xacro"/> -->
+  <!-- <xacro:table ns="panda" rpy="0 0 0" xyz="0.68 0 0.0375" connected_to="panda_link0"/> -->
 </robot>

Commit message: Update URDF to include hose

File: mercury/_pybullet/robots/franka_panda/panda_reorient.urdf (robot description, URDF)
Before this commit: robot panda, 11 links, 10 joints
Links:
- link tipLink: geometry collision cylinder length=0.18 radius=0.02; visual cylinder length=0.11 radius=0.02

File: ros/mercury_panda/robots/include/suction_gripper.xacro (robot description, xacro)
@@ -38,7 +38,7 @@
       <collision>
         <geometry>
-          <cylinder length="0.11" radius="0.02"/>
+          <cylinder length="0.18" radius="0.02"/>
         </geometry>
-        <origin xyz="0 0 -0.055"/>
+        <origin xyz="0 0 -0.09"/>
       </collision>
     </link>

Commit message: Add drl to mercury/_pybullet/robots/franka_panda

File: mercury/_pybullet/robots/franka_panda/panda_reorient.urdf (robot description, URDF)
Before this commit: robot panda, 11 links, 10 joints
Links:
- link panda_suction_gripper: geometry collision mesh filename=package://drl/meshes/collision/suction_mount.obj; visual mesh filename=package://drl/meshes/visual/suction_mount.obj

File: mercury/_pybullet/robots/franka_panda/panda_reorient.urdf.xacro (robot description, xacro)
@@ -2,5 +2,5 @@
 <robot xmlns:xacro="http://www.ros.org/wiki/xacro" name="panda">
   <xacro:include filename="panda_arm.urdf"/>
-  <xacro:include filename="$(find mercury_panda)/robots/include/suction_gripper.xacro"/>
+  <xacro:include filename="$(find mercury_panda)/robots/drl/suction.xacro"/>
   <xacro:suction_gripper ns="panda" rpy="${pi} 0 ${-pi/4}" xyz="0 0 0.0065" connected_to="panda_link8"/>
   <!-- <xacro:include filename="$(find mercury_panda)/robots/include/table.xacro"/> -->
