Commit message: Update panda_drl.urdf and panda_suction.urdf with new panda_arm.urdf

File: mercury/_pybullet/robots/franka_panda/panda_drl.urdf (robot description, URDF)
Before this commit: robot panda, 11 links, 10 joints
Joints:
- joint panda_joint1: limit lower=-2.9671 upper=2.9671 effort=87 velocity=2.1750 -> lower=-2.8973 upper=2.8973 effort=87 velocity=2.1750
- joint panda_joint2: limit lower=-1.8326 upper=1.8326 effort=87 velocity=2.1750 -> lower=-1.7628 upper=1.7628 effort=87 velocity=2.1750
- joint panda_joint3: limit lower=-2.9671 upper=2.9671 effort=87 velocity=2.1750 -> lower=-2.8973 upper=2.8973 effort=87 velocity=2.1750
- joint panda_joint4: limit lower=-3.1416 upper=0.0 effort=87 velocity=2.1750 -> lower=-3.0718 upper=-0.0698 effort=87 velocity=2.1750
- joint panda_joint5: limit lower=-2.9671 upper=2.9671 effort=12 velocity=2.6100 -> lower=-2.8973 upper=2.8973 effort=12 velocity=2.6100
- joint panda_joint6: limit lower=-0.0873 upper=3.8223 effort=12 velocity=2.6100 -> lower=-0.0175 upper=3.7525 effort=12 velocity=2.6100
- joint panda_joint7: limit lower=-2.9671 upper=2.9671 effort=12 velocity=2.6100 -> lower=-2.8973 upper=2.8973 effort=12 velocity=2.6100

File: mercury/_pybullet/robots/franka_panda/panda_suction.urdf (robot description, URDF)
Before this commit: robot panda, 13 links, 12 joints
Joints:
- joint panda_joint1: limit lower=-2.9671 upper=2.9671 effort=87 velocity=2.1750 -> lower=-2.8973 upper=2.8973 effort=87 velocity=2.1750
- joint panda_joint2: limit lower=-1.8326 upper=1.8326 effort=87 velocity=2.1750 -> lower=-1.7628 upper=1.7628 effort=87 velocity=2.1750
- joint panda_joint3: limit lower=-2.9671 upper=2.9671 effort=87 velocity=2.1750 -> lower=-2.8973 upper=2.8973 effort=87 velocity=2.1750
- joint panda_joint4: limit lower=-3.1416 upper=0.0 effort=87 velocity=2.1750 -> lower=-3.0718 upper=-0.0698 effort=87 velocity=2.1750
- joint panda_joint5: limit lower=-2.9671 upper=2.9671 effort=12 velocity=2.6100 -> lower=-2.8973 upper=2.8973 effort=12 velocity=2.6100
- joint panda_joint6: limit lower=-0.0873 upper=3.8223 effort=12 velocity=2.6100 -> lower=-0.0175 upper=3.7525 effort=12 velocity=2.6100
- joint panda_joint7: limit lower=-2.9671 upper=2.9671 effort=12 velocity=2.6100 -> lower=-2.8973 upper=2.8973 effort=12 velocity=2.6100

Commit message: Update URDF

File: mercury/_pybullet/robots/franka_panda/panda_drl.urdf (robot description, URDF)
Before this commit: robot panda, 11 links, 10 joints
Links:
- link tipLink: geometry collision cylinder length=0.16 radius=0.018; visual cylinder length=0.10 radius=0.018
Joints:
- joint panda_suction_mount_to_cup_joint: origin xyz=0.072 0 -0.09 rpy=3.14159265359 0 0 -> xyz=0.072 0 -0.08 rpy=3.14159265359 0 0

File: ros/mercury_panda/robots/drl/suction.xacro (robot description, xacro)
@@ -31,14 +31,14 @@
       <visual>
         <geometry>
-          <cylinder length="0.11" radius="0.02"/>
+          <cylinder length="0.10" radius="0.018"/>
         </geometry>
-        <origin xyz="0 0 -0.055"/>
+        <origin xyz="0 0 -0.05"/>
         <material name="green"/>
       </visual>
       <collision>
         <geometry>
-          <cylinder length="0.18" radius="0.02"/>
+          <cylinder length="0.16" radius="0.018"/>
         </geometry>
-        <origin xyz="0 0 -0.09"/>
+        <origin xyz="0 0 -0.08"/>
       </collision>
     </link>
@@ -46,5 +46,5 @@
       <parent link="${ns}_suction_gripper"/>
       <child link="tipLink"/>
-      <origin xyz="0.072 0 -0.09" rpy="${pi} 0 0"/>
+      <origin xyz="0.072 0 -0.08" rpy="${pi} 0 0"/>
     </joint>
   </xacro:macro>

Commit message: Cleanup file path for URDF

File: mercury/_pybullet/robots/franka_panda/panda_drl.urdf (robot description, URDF)
Before this commit: robot panda, 11 links, 10 joints
Links:
- link panda_suction_gripper: geometry collision mesh filename=package://mercury_panda/robots/drl/meshes/collision/suction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; visual mesh filename=package://mercury_panda/robots/drl/meshes/visual/suction_mo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
Joints:
- joint panda_suction_gripper_joint: origin xyz=0 0 0.0065 rpy=3.14159265359 0 -0.785398163397 -> xyz=0 0 0.0065 rpy=3.141592653589793 0 -0.7853981633974483
- joint panda_suction_mount_to_cup_joint: origin xyz=0.072 0 -0.08 rpy=3.14159265359 0 0 -> xyz=0.072 0 -0.08 rpy=3.141592653589793 0 0

File: mercury/_pybullet/robots/franka_panda/panda_drl.urdf.xacro (robot description, xacro)
@@ -4,5 +4,3 @@
   <xacro:include filename="$(find mercury_panda)/robots/drl/suction.xacro"/>
   <xacro:suction_gripper ns="panda" rpy="${pi} 0 ${-pi/4}" xyz="0 0 0.0065" connected_to="panda_link8"/>
-  <!-- <xacro:include filename="$(find mercury_panda)/robots/include/table.xacro"/> -->
-  <!-- <xacro:table ns="panda" rpy="0 0 0" xyz="0.68 0 0.0375" connected_to="panda_link0"/> -->
 </robot>
