Commit message: safepicking/_pybullet/: mercury -> safepicking

File: safepicking/_pybullet/data/franka_panda/panda_drl.urdf (robot description, URDF)
Before this commit: robot panda, 11 links, 10 joints
Links:
- link panda_suction_gripper: geometry collision mesh filename=package://safepicking_ros/robots/drl/meshes/collision/sucti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; visual mesh filename=package://safepicking_ros/robots/drl/meshes/visual/suction_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

File: safepicking/_pybullet/data/franka_panda/panda_drl.urdf.xacro (robot description, xacro)
@@ -2,5 +2,5 @@
 <robot xmlns:xacro="http://www.ros.org/wiki/xacro" name="panda">
   <xacro:include filename="panda_arm.urdf"/>
-  <xacro:include filename="$(find mercury_ros)/robots/drl/suction.xacro"/>
+  <xacro:include filename="$(find safepicking_ros)/robots/drl/suction.xacro"/>
   <xacro:suction_gripper ns="panda" rpy="${pi} 0 ${-pi/4}" xyz="0 0 0.0065" connected_to="panda_link8"/>
 </robot>
