Commit message: ros/src/safepicking_ros: mercury -> safepicking

File: ros/src/safepicking_ros/robots/drl/suction.xacro (robot description, xacro)
@@ -18,5 +18,5 @@
       <visual>
         <geometry>
-          <mesh filename="package://mercury_ros/robots/drl/meshes/visual/suction_mount.obj"/>
+          <mesh filename="package://safepicking_ros/robots/drl/meshes/visual/suction_mount.obj"/>
         </geometry>
         <material name="black"/>
@@ -24,5 +24,5 @@
       <collision>
         <geometry>
-          <mesh filename="package://mercury_ros/robots/drl/meshes/collision/suction_mount.obj"/>
+          <mesh filename="package://safepicking_ros/robots/drl/meshes/collision/suction_mount.obj"/>
         </geometry>
       </collision>

File: ros/src/safepicking_ros/robots/panda_drl.urdf.xacro (robot description, xacro)
@@ -2,5 +2,5 @@
 <robot xmlns:xacro="http://www.ros.org/wiki/xacro" name="panda">
   <xacro:include filename="$(find franka_description)/robots/panda_arm.urdf.xacro"/>
-  <xacro:include filename="$(find mercury_ros)/robots/drl/suction.xacro"/>
+  <xacro:include filename="$(find safepicking_ros)/robots/drl/suction.xacro"/>
   <xacro:suction_gripper ns="panda" rpy="${pi} 0 ${-pi/4}" xyz="0 0 0.0065" connected_to="panda_link8"/>
 </robot>
